Commit message: Added meshes & measures for urdf description

File: urdf/robot_view.urdf (robot description, URDF)
Before this commit: robot wheels, 6 links, 5 joints
Links:
- link back_left_wheel_link: mass 0.01 -> 1.6; geometry collision cylinder length=${WW} radius=${WR}; visual mesh filename=package://pai/meshes/wheel.dae
- link back_right_wheel_link: mass 0.01 -> 1.6; geometry collision cylinder length=${WW} radius=${WR}; visual mesh filename=package://pai/meshes/wheel.dae
- link base_link: geometry collision box size=${BL} ${BW} ${BH}; visual mesh filename=package://pai/meshes/box.dae
- link front_left_wheel_link: mass 0.01 -> 1.6; geometry collision cylinder length=${WW} radius=${WR}; visual mesh filename=package://pai/meshes/wheel.dae
- link front_right_wheel_link: mass 0.01 -> 1.6
Joints:
- joint back_left_wheel_joint: origin xyz=${-L} ${BW/2 + WW/2} ${WR} rpy=$(eval pi/2) 0.0 0.0 -> xyz=${-L} ${BW/2 + WW/2} ${WR} rpy=${pi/2} 0.0 0.0
- joint back_right_wheel_joint: origin xyz=${-L} ${-BW/2 - WW/2} ${WR} rpy=$(eval -pi/2) 0.0 0.0 -> xyz=${-L} ${-BW/2 - WW/2} ${WR} rpy=${-pi/2} 0.0 0.0
- joint front_left_wheel_joint: origin xyz=${L} ${BW/2 + WW/2} ${WR} rpy=$(eval pi/2) 0.0 0.0 -> xyz=${L} ${BW/2 + WW/2} ${WR} rpy=${pi/2} 0.0 0.0
- joint front_right_wheel_joint: origin xyz=${L} ${-BW/2 - WW/2} ${WR} rpy=$(eval -pi/2) 0.0 0.0 -> xyz=${L} ${-BW/2 - WW/2} ${WR} rpy=${-pi/2} 0.0 0.0

Commit message: modify urdf

File: urdf/robot_view.urdf (robot description, URDF)
Before this commit: robot wheels, 6 links, 5 joints
Links:
- link front_right_wheel_link: geometry collision cylinder length=${WW} radius=${WR}; visual mesh filename=package://pai/meshes/wheel.dae

Commit message: modify urdf with xacro macro

File: urdf/robot_view.urdf (robot description, URDF)
Before this commit: robot wheels, 6 links, 5 joints
Links:
- removed link back_left_wheel_link
- removed link back_right_wheel_link
- removed link front_left_wheel_link
- removed link front_right_wheel_link
- link base_link: mass None -> 1.0
Joints:
- removed joint back_left_wheel_joint
- removed joint back_right_wheel_joint
- removed joint front_left_wheel_joint
- removed joint front_right_wheel_joint
