Commit message: add rqt dependencies

File: urdf/robot.urdf (robot description, URDF)
Before this commit: robot ugv, 2 links, 1 joints
Links:
- link base_link: geometry collision box size=${BL} ${BW-0.01} ${BH}; visual mesh filename=package://pai/meshes/box.dae

Commit message: Fix simulation and comment velocity limits in kinematic model

File: urdf/robot.urdf (robot description, URDF)
Before this commit: robot ugv, 2 links, 1 joints
Links:
- link base_link: mass 1.0 -> 30.0
